File: MPad2040_V1.kicad_pcb (KiCad board)
At the start: 2 copper layers, 81.3 x 128.9 mm, 94 parts, among them J1 DNP, J2 USB_C_Receptacle_USB2.0, SW1 SW_E1, SW10 SW_8, SW11 SW_9, SW12 SW_+2u, SW13 SW_4, SW14 SW_5, SW15 SW_6, SW16 SW_1, SW17 SW_2, SW18 SW_3, SW19 SW_ENTER-2u, SW2 SW_E2, SW20 SW_0-2u, SW21 SW_dot, SW22 SW_-1u, SW23 SW_+1u, SW24 SW_R4_1u, SW25 SW_R3_1u, SW26 SW_00-1u, SW27 SW_0-1u, SW28 ~{RESET}, SW29 ~{USB_boot}, SW3 SW_E3, SW4 SW_E4, SW5 SW_NUM, SW6 SW_/, SW7 SW_*, SW8 SW_-, SW9 SW_7, U1 SC09087_functional, U2 AMS1117-3.3, U3 W25Q16JVSSIQ, Y1 12MHz

Commit message: updates
Parts:
- removed the G*** at (147.5, 96.2)
- removed REF**: OSHW-Logo2_7.3x6mm_SilkScreen, Symbol:OSHW-Logo2_7.3x6mm_SilkScreen
- added G***: LOGO, MPad2040:Saturn3, B.Cu at (131.5, 58.3)
- moved R5 2.06 mm to (167.5, 47.2)
- moved R6 2.06 mm to (166.0, 47.2)
- moved C4 1.53 mm to (167.5, 50.5), turned to 90 degrees
- moved C13 1.35 mm to (164.7, 50.4)
- moved C8 1.35 mm to (165.6, 50.4)
- moved C15 0.37 mm to (164.8, 61.2)
- moved C5 0.37 mm to (165.8, 61.2)
- moved C11 0.13 mm to (168.9, 51.6)
Connections:
- C13 pad 1: +3V3 -> /VREG_VOUT
- C5 pad 1: +3V3 -> /VREG_VOUT
- U1 pad 23: +3V3 -> /VREG_VOUT
- U1 pad 50: +3V3 -> /VREG_VOUT
Routing:
- net /VREG_VOUT: track 2.97 -> 16.0 mm
- net +3V3: track 151.4 -> 147.8 mm
- net /USB_D+: track 13.0 -> 10.9 mm
- net /2040_D-: track 2.81 -> 4.89 mm
- net /2040_D+: track 2.81 -> 4.88 mm
- net /USB_D-: track 13.0 -> 11.0 mm
Other:
- board text added: "*"
- board text added: "+"
- board text added: ","
- board text added: "-"
- board text added: "/"
- board text added: "0"
- board text added: "1"
- board text added: "2"
- board text added: "3"
- board text added: "4"
- board text added: "5"
- board text added: "6"
- board text added: "7"
- board text added: "8"
- board text added: "9"
- board text added: "E1"
- board text added: "E2"
- board text added: "E3"
- board text added: "E4"
- board text added: "Enter"
- board text added: "NumLock"
