File: MPad2040_V1.kicad_sch (KiCad schematic)
At the start: 91 parts, among them J1 DNP, J2 USB_C_Receptacle_USB2.0, SW1 SW_E1, SW10 SW_8, SW11 SW_9, SW12 SW_+2u, SW13 SW_4, SW14 SW_5, SW15 SW_6, SW16 SW_1, SW17 SW_2, SW18 SW_3, SW19 SW_ENTER-2u, SW2 SW_E2, SW20 SW_0-2u, SW21 SW_dot, SW22 SW_-1u, SW23 SW_+1u, SW24 SW_R4_1u, SW25 SW_R3_1u, SW26 SW_00-1u, SW27 SW_0-1u, SW28 ~{RESET}, SW29 ~{USB_boot}, SW3 SW_E3, SW4 SW_E4, SW5 SW_NUM, SW6 SW_/, SW7 SW_*, SW8 SW_-, SW9 SW_7, U1 SC09087_functional, U2 AMS1117-3.3, U3 W25Q16JVSSIQ, Y1 12MHz

Commit message: updates
Connections:
- net +3V3: no longer C13.1, C5.1, U1.23 (DVDD), U1.50 (DVDD)
- net VREG_VOUT: now also C13.1, C5.1, U1.23 (DVDD), U1.50 (DVDD)
Other:
- moved on the sheet: C13, C14, C15, C16, C6, C7, C8

Commit message: Version 1.1 finalized
Parts:
- FB1: value 600R@100MHz -> 220R@100MHz
- J2: footprint MPad2040:USB_C_Receptacle_GCT_USB4085 -> MPad2040:USB_C_Receptacle_Palconn_UTC16-G
- R5, R6: footprint Resistor_SMD:R_0603_1608Metric -> Resistor_SMD:R_0402_1005Metric
Other:
- note removed: "ATH - má fækka þéttum í neyð"
Changed lines of the file:
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@@
     (effects (font (size 1.27 1.27)) (justify left bottom))
-  )
-  (text "ATH - má fækka\nþéttum í neyð" (at 185.42 88.9 0)
-    (effects (font (size 2 2) (thickness 0.4) bold) (justify left bottom))
   )
   (text "A 10k resistor can be placed here if\nnecessary, to insure that CS is high\nduring a short period of time when the\nRP2040 is powered up (in which the\nstate of QSPI_SS_N can't be guaranteed)"
@@
   (symbol (lib_id "power:+3.3V") (at 248.92 68.58 0) (unit 1)
     (in_bom yes) (on_board yes) (dnp no)
-    (property "Reference" "#PWR?" (at 248.92 72.39 0)
+    (property "Reference" "#PWR0102" (at 248.92 72.39 0)
       (effects (font (size 1.27 1.27)) hide)
     )
@@
       (project "MPad2040_V1"
         (path "/e63e39d7-6ac0-4ffd-8aa3-1841a4541b55"
-          (reference "#PWR?") (unit 1)
+          (reference "#PWR0102") (unit 1)
         )
       )
@@
       (effects (font (size 1.27 1.27)))
     )
-    (property "Footprint" "Resistor_SMD:R_0603_1608Metric" (at 175.26 162.56 0)
+    (property "Footprint" "Resistor_SMD:R_0402_1005Metric" (at 175.26 162.56 0)
       (effects (font (size 1.27 1.27)) hide)
     )
@@
       (effects (font (size 1.27 1.27)))
     )
-    (property "Footprint" "MPad2040:USB_C_Receptacle_GCT_USB4085" (at 87.63 60.96 0)
+    (property "Footprint" "MPad2040:USB_C_Receptacle_Palconn_UTC16-G" (at 87.63 60.96 0)
       (effects (font (size 1.27 1.27)) hide)
     )
@@
       (effects (font (size 1.27 1.27)))
     )
-    (property "Footprint" "Resistor_SMD:R_0603_1608Metric" (at 175.26 165.1 0)
+    (property "Footprint" "Resistor_SMD:R_0402_1005Metric" (at 175.26 165.1 0)
       (effects (font (size 1.27 1.27)) hide)
     )
@@
   (symbol (lib_id "Device:FerriteBead_Small") (at 124.46 45.72 90) (unit 1)
     (in_bom yes) (on_board yes) (dnp no) (fields_autoplaced)
-    (property "Reference" "FB1" (at 124.4219 39.37 90)
-      (effects (font (size 1.27 1.27)))
-    )
-    (property "Value" "600R@100MHz" (at 124.4219 41.91 90)
+    (property "Reference" "FB1" (at 124.4219 40.64 90)
+      (effects (font (size 1.27 1.27)))
+    )
+    (property "Value" "220R@100MHz" (at 124.4219 43.18 90)
       (effects (font (size 1.27 1.27)))
     )
@@
   (symbol (lib_id "power:+3.3V") (at 205.74 59.69 0) (unit 1)
     (in_bom yes) (on_board yes) (dnp no)
-    (property "Reference" "#PWR?" (at 205.74 63.5 0)
+    (property "Reference" "#PWR0103" (at 205.74 63.5 0)
       (effects (font (size 1.27 1.27)) hide)
     )
@@
       (project "MPad2040_V1"
         (path "/e63e39d7-6ac0-4ffd-8aa3-1841a4541b55"
-          (reference "#PWR?") (unit 1)
-        )
-      )
+          (reference "#PWR0103") (unit 1)
+        )
+      )

Commit message: Fixes for V1.1
Parts:
- R4, R7, R8: footprint Resistor_SMD:R_0603_1608Metric -> Resistor_SMD:R_0402_1005Metric
Changed lines of the file:
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@@
       (effects (font (size 1.27 1.27)) (justify left))
     )
-    (property "Footprint" "Resistor_SMD:R_0603_1608Metric" (at 172.72 53.34 0)
+    (property "Footprint" "Resistor_SMD:R_0402_1005Metric" (at 172.72 53.34 0)
       (effects (font (size 1.27 1.27)) hide)
     )
@@
       (effects (font (size 1.27 1.27)))
     )
-    (property "Footprint" "Resistor_SMD:R_0603_1608Metric" (at 233.68 210.82 0)
+    (property "Footprint" "Resistor_SMD:R_0402_1005Metric" (at 233.68 210.82 0)
       (effects (font (size 1.27 1.27)) hide)
     )
@@
       (effects (font (size 1.27 1.27)))
     )
-    (property "Footprint" "Resistor_SMD:R_0603_1608Metric" (at 182.88 137.16 0)
-      (effects (font (size 1.27 1.27)) hide)
-    )
+    (property "Footprint" "Resistor_SMD:R_0402_1005Metric" (at 182.88 137.16 0)
+      (effects (font (size 1.27 1.27)) hide)
+    )
